File: dogbone.kicad_pcb (KiCad board)
At the start: 2 copper layers, 4.8 x 23 mm, 12 parts, among them M1 THRU_HOLE_PAD, M10 THRU_HOLE_PAD, M11 THRU_HOLE_PAD, M12 THRU_HOLE_PAD, M2 THRU_HOLE_PAD, M3 THRU_HOLE_PAD, M4 THRU_HOLE_PAD, M5 THRU_HOLE_PAD, M6 THRU_HOLE_PAD, M7 THRU_HOLE_PAD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

Commit message: reverted baseplate back to all on top, designed to flip over, and solder from the component side. dogbone bottom changed so one end has three prongs
Parts:
- moved M2 1.15 mm to (88.5, 70.2)
- moved M6 1.15 mm to (88.5, 70.2)
- moved M10 0.15 mm to (86.6, 70.2)
- moved M11 0.15 mm to (90.4, 70.2)
- moved M12 0.15 mm to (90.4, 70.2)
- moved M3 0.15 mm to (86.6, 70.2)
Routing:
- net /SIN: track 20.0 -> 21.1 mm
- net /COS: track 20.0 -> 21.1 mm
Other:
- board size 4.8 x 23 mm -> 4.8 x 23.1 mm
